File: hardware/OAS-core/OAS-core.kicad_sch (KiCad schematic)
At the start: 8 parts, among them J1 Micro_SD_Card, J2 PROG, J3 MSC, J4 Conn_01x02_Pin, U1 ESP32-WROOM-32, U2 TPS2116DRL/TPS2117, U3 TPS54336ADDA, U5 TPS563202DRLR

Commit message: PSU
Parts:
- removed U3: TPS54336ADDA, Package_SO:TI_SO-PowerPAD-8_ThermalVias, symbol Regulator_Switching:TPS54336ADDA
- added C1: 220p, Capacitor_SMD:C_0402_1005Metric, symbol Device:C
- added C2: 220u, Capacitor_SMD:CP_Elec_8x10.5, symbol Device:C_Polarized_US
- added C3: 1u, Capacitor_SMD:C_0402_1005Metric, symbol Device:C
- added C4: 10n, Capacitor_SMD:C_0402_1005Metric, symbol Device:C
- added C5: 220u, Capacitor_SMD:CP_Elec_6.3x5.9, symbol Device:C_Polarized_US
- added D1: D_Schottky, Diode_SMD:D_SMA, symbol Device:D_Schottky
- added F1: 1.5A, Resistor_SMD:R_0603_1608Metric, symbol Device:Fuse
- added L1: PSPHAQ127-180M, Inductor_SMD:L_12x12mm_H8mm, symbol Device:L
- added R1: 220K, Resistor_SMD:R_0402_1005Metric, symbol Device:R
- added R2: 20K, Resistor_SMD:R_0402_1005Metric, symbol Device:R
- added R3: 10K, Resistor_SMD:R_0402_1005Metric, symbol Device:R
- added R4: 6.8K, Resistor_SMD:R_0402_1005Metric, symbol Device:R
- added R5: 3.3k, Resistor_SMD:R_0402_1005Metric, symbol Device:R
- added R6: 10k, Resistor_SMD:R_0402_1005Metric, symbol Device:R
- added R7: 0, Resistor_SMD:R_0402_1005Metric, symbol Device:R
- added U4: TPS26600, Package_SO:HTSSOP-16-1EP_4.4x5mm_P0.65mm_EP3.4x5mm_Mask2.46x2.31mm_ThermalVias, symbol oas:TPS26601
- added U6: TPS5430DDA, Package_SO:TI_SO-PowerPAD-8_ThermalVias, symbol Regulator_Switching:TPS5430DDA
- J4: value Conn_01x02_Pin -> XT30PW-M; footprint (none) -> Connector_AMASS:AMASS_XT30PW-M_1x02_P2.50mm_Horizontal
- U2: value TPS2116DRL/TPS2117 -> TPS2116DRL; LCSC (none) -> C3235557
Connections:
- net GND: now reaches J4.1 (Pin_1)
- net GND: now also C2.2, C3.2, C5.2, D1.2 (A), R5.2, U4.9 (GND), U6.6 (GND), U6.9 (GNDPAD)
- net at J4.2 (Pin_2): now also F1.2
- new net: R5.1, R6.2, U6.4 (VSENSE)
- new net: C3.1, R7.2, U6.7 (VIN)
- new net: C4.1, U6.1 (BOOT)
- new net: C4.2, D1.1 (K), L1.1, U6.8 (PH)
- new net: C1.1, U4.12 (dVdT)
- new net: C1.2, R3.2, R4.2, U4.17 (PAD), U4.8 (RTN)
- new net: F1.1, R1.1, U4.1 (IN), U4.2 (IN)
- new net: R4.1, U4.11 (I_{LIM})
- new net: R1.2, R2.1, U4.3 (UVLO)
- new net: R2.2, R3.1, U4.5 (OVP)
- new net +5_{VIN}: C5.1, L1.2, R6.1
- new net +VIN_{PROT}: C2.1, R7.1, U4.15 (OUT), U4.16 (OUT)
- new net pgood: U4.14 (~{FLT}), U6.5 (EN)
- no-connect marks 0 -> 3
Other:
- removed sheet vin_prot
- note added: "Criteria: - circuit breaker mode - auto-retry - 1.75A OCP - 29.7 OVP - 9.9 UVLO - 220uF load capacitance"
- note added: "VIN -> 5V"
- note added: "https://www.ti.com/tool/PMP10737 TPS2660 DPS1133 LM7480"
- note removed: "https://naturesgenerator.com/blogs/news/lead-acid-battery-voltage-chart"
- moved on the sheet: J3, J4, U2, U5

Commit message: PSU
Parts:
- added Q1, Q2: PMOS, symbol Simulation_SPICE:PMOS
- added R8: R, symbol Device:R
- added U3: TPS2116DRL, Package_TO_SOT_SMD:SOT-583-8, symbol Power_Management:TPS2116DRL
- added U7: LM66100DCK, Package_TO_SOT_SMD:SOT-363_SC-70-6, symbol Power_Management:LM66100DCK
Connections:
- net +5_{VIN} is gone; now on net +5V_{in}: C5.1, L1.2, R6.1
- net GND: now also U2.1 (GND), U2.4 (PR1), U2.5 (MODE)
- net at J3.1 (VBUS): now also U2.6 (VIN2)
- net +5V_{ext}: now reaches U2.2 (VOUT), U2.7 (VOUT)
- net +5V_{ext}: now also R8.1
- net +5V_{in}: now reaches U2.3 (VIN1)
- net at U2.8 (ST): now also R8.2
- net +VIN_{PROT} renamed +V_{in}
- new net: U3.2 (VOUT), U3.7 (VOUT)
- new net +3V3_{out}: Q2.3 (S)
- new net +5V_{out}: Q1.3 (S)
Other:
- note added: "PSU MDOES Input | +V_{out} ---------------------------- VIN | ACTIVE USB_PROG | ACTIVE USB_MSC | INACTIVE BATT | INACTIVE"
- moved on the sheet: C5, J2, J3, R5, R6, U2, U5

Commit message: PSU Mux
Parts:
- removed R8: R, symbol Device:R
- removed U2: TPS2116DRL, Package_TO_SOT_SMD:SOT-583-8, symbol Power_Management:TPS2116DRL
- removed U7: LM66100DCK, Package_TO_SOT_SMD:SOT-363_SC-70-6, symbol Power_Management:LM66100DCK
- added D2, D3, D4, D5: SS54, Diode_SMD:D_SMA, symbol Device:D_Schottky
Connections:
- net VMUX2: now reaches J3.1 (VBUS)
- net VMUX1: now reaches J2.1 (VBUS)
- new net: D2.1 (K), D3.1 (K), D4.1 (K), D5.1 (K)
Other:
- moved on the sheet: J2, J3, Q1, Q2, U3, U5

Commit message: Mux
Parts:
- removed D2, D3, D4, D5: SS54, Diode_SMD:D_SMA, symbol Device:D_Schottky
Connections:
- net +5V_{in} renamed 5V_{IN}
- net +V_{in}: no longer names the net of C2.1, R7.1, U4.15 (OUT), U4.16 (OUT)
- net VMUX1 renamed 5V_{USB,PROG}
- net VMUX2 renamed 5V_{USB,MSC}
Other:
- added sheet Power Mux (power_mux.kicad_sch)

Commit message: PSU
Parts:
- removed U5: TPS563202DRLR, Package_TO_SOT_SMD:SOT-563, symbol Regulator_Switching:TPS563202S
- added L2: L, symbol Device:L
- added U2: LM66200, Package_SON:Texas_R-PUSON-N8_USON-8-1EP_1.6x2.1mm_P0.5mm_EP0.4x1.7mm, symbol oas:LM66200
- added U7: TPS63000, Package_SON:Texas_DRC0010J_ThermalVias, symbol Regulator_Switching:TPS63000
Connections:
- new net: U2.1 (GND), U2.5 (GND)
- new net: U2.2 (VOUT), U2.7 (VOUT)
- new net: U7.11 (PGND), U7.3 (PGND)
- new net: L2.2, U7.2 (L2)
- new net: L2.1, U7.4 (L1)
Other:
- removed sheet Power Mux
- note added: "MCU powered from batt 2V7-4V2 OR 5V"

Commit message: MCU PSU spec + impl
Parts:
- removed U1: ESP32-WROOM-32, RF_Module:ESP32-WROOM-32, symbol RF_Module:ESP32-WROOM-32
- removed U2: LM66200, Package_SON:Texas_R-PUSON-N8_USON-8-1EP_1.6x2.1mm_P0.5mm_EP0.4x1.7mm, symbol oas:LM66200
- removed U3: TPS2116DRL, Package_TO_SOT_SMD:SOT-583-8, symbol Power_Management:TPS2116DRL
- removed U7: TPS63000, Package_SON:Texas_DRC0010J_ThermalVias, symbol Regulator_Switching:TPS63000
- added BT2: Battery_Cell, Connector_JST:JST_PH_B2B-PH-SM4-TB_1x02-1MP_P2.00mm_Vertical, symbol Device:Battery_Cell
- added C6, C7: 10u, Capacitor_SMD:C_0805_2012Metric, symbol Device:C
- added C8: 1u, Capacitor_SMD:C_0402_1005Metric, symbol Device:C
- added D2, D3: D_Schottky, symbol Device:D_Schottky
- added R10, R8, R9: 47K, Resistor_SMD:R_0402_1005Metric, symbol Device:R
- added R11: 10k, Resistor_SMD:R_0402_1005Metric, symbol Device:R
- added R12: 100, Resistor_SMD:R_0402_1005Metric, symbol Device:R
- added U1: ESP32-S3-MINI-1, RF_Module:ESP32-S2-MINI-1, symbol RF_Module:ESP32-S3-MINI-1
- added U2: MT3406, Package_TO_SOT_SMD:SOT-23-5, symbol oas:MT3406
- added U3: LM66200, Package_TO_SOT_SMD:SOT-583-8, symbol oas:LM66200
- added U5: CH340X, Package_SO:MSOP-10_3x3mm_P0.5mm, symbol Interface_USB:CH340X
- added U7: TP4054, Package_TO_SOT_SMD:TSOT-23-5, symbol Battery_Management:LTC4054ES5-4.2
- added U8: DW02, Package_TO_SOT_SMD:SOT-23-5, symbol oas:DW02
- J1: footprint (none) -> Connector_Card:microSD_HC_Hirose_DM3AT-SF-PEJM5; LCSC (none) -> C114218
- J2, J3: footprint (none) -> Connector_USB:USB_B_OST_USB-B1HSxx_Horizontal
- L2: value L -> 2.2u; footprint (none) -> Inductor_SMD:L_1008_2520Metric; LCSC (none) -> C5156791
Connections:
- net GND: now also J2.4 (GND), J2.5 (Shield), J3.4 (GND), J3.5 (Shield), C6.2, C7.2, C8.2, R10.2, R11.2, U1.1 (GND), U1.2 (GND), U1.42 (GND), U1.43 (GND), U1.46 (GND), U1.47 (GND), U1.48 (GND), U1.49 (GND), U1.50 (GND), U1.51 (GND), U1.52 (GND), U1.53 (GND), U1.54 (GND), U1.55 (GND), U1.56 (GND), U1.57 (GND), U1.58 (GND), U1.59 (GND), U1.60 (GND), U1.61 (GND), U1.62 (GND), U1.63 (GND), U1.64 (GND), U1.65 (GND), U2.2 (GND), U3.1 (GND), U3.4 (~{ON}), U3.5 (GND), U7.2 (GND), U8.4 (VSS), U8.5 (VSS)
- net RTN: now reaches C1.2, R3.2, R4.2, U4.17 (PAD), U4.8 (RTN)
- net +3.3V_{core}: now reaches L2.2
- net +3.3V_{core}: now also C7.1, R9.1
- net at L2.1: now also U2.3 (SW)
- net 5V_{IN} renamed +5V
- net +5V: now also C8.1, D2.1 (K), D3.1 (K), U3.3 (VIN1), U7.4 (V_{CC})
- net 5V_{USB,MSC}: no longer names the net of J3.1 (VBUS)
- net 5V_{USB,MSC}: now also D3.2 (A)
- net 5V_{USB,PROG}: no longer names the net of J2.1 (VBUS)
- net 5V_{USB,PROG}: now also D2.2 (A)
- new net: R11.1, U7.1 (~{CHRG})
- new net: C6.1, R8.1, U2.1 (EN), U2.4 (VIN), U3.2 (VOUT), U3.7 (VOUT)
- new net: BT2.2 (-), U8.2 (B-)
- new net: R12.2, U8.3 (VDD)
- new net: R10.1, R9.2, U2.5 (FB)
- new net +BATT: BT2.1 (+), R12.1, U3.6 (VIN2), U7.3 (BAT)
- new net V_{core, source}: R8.2, U3.8 (ST)
- no-connect marks 3 -> 4
Other:
- note added: "Battery + Charging (100mA) + Protection"
- note added: "MCU PSU (UPS)"
- note removed: "5->3v3"
- note removed: "MCU powered from batt 2V7-4V2 OR 5V"
- note removed: "PSU MDOES Input | +V_{out} ---------------------------- VIN | ACTIVE USB_PROG | ACTIVE USB_MSC | INACTIVE BATT | INACTIVE"
- moved on the sheet: J1
